Commit message: Update to large formation experiences

File: uned_khepera_description/urdf/khepera_simple.urdf (robot description, URDF)
Before this commit: robot khepera, 3 links, 2 joints
Links:
- removed link chassis
- removed link left_wheel
- link base_link: mass None -> 0.5; geometry collision mesh filename=package://uned_khepera_description/meshes/files/Empty_robot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 scale=1.0 1.0 1.0; visual mesh filename=package://uned_khepera_description/meshes/files/Empty_robot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 scale=1.0 1.0 1.0
Joints:
- removed joint base_link_joint
- removed joint left_wheel_joint
