Commit message: refactor: rename uned_khepera_gazebo -> uned_kheperaiv_gazebo, merge uned_khepera_description into uned_kheperaiv_config
Per your direction: uned_khepera_gazebo renamed for naming consistency with
the rest of the repo (uned_kheperaiv_*). uned_khepera_description didn't
make sense as a standalone package -- merged into uned_kheperaiv_config
(urdf/, meshes/, the URDF-generation CMake macro from its CMakeLists.txt,
launch/urdf_visualize.launch.py, rviz/urdf_simple.rviz, src/replace.py),
same call as uned_crazyflie_common -> uned_crazyflie_driver in the
Crazyflie repo.

Updated every real reference to the old package (get_package_share_directory
calls in the two Gazebo formation launch files, package:// mesh URIs in the
URDF files, urdf_visualize.launch.py's package_description variable, and
the RViz 'Description File' absolute paths in default.rviz/
formation_distance_four.rviz -- those still hardcode Francisco's own local
clone path, a pre-existing portability issue not introduced here, only the
package-name segment was corrected).

Verified with a real colcon build: both packages build clean, the 40
generated kheperaXX.urdf + the 3 source urdf files + all mesh files install
correctly under uned_kheperaiv_config's share directory, replace.py
installs as an executable script.

File: uned_kheperaiv_config/urdf/khepera.urdf (robot description, URDF)
Before this commit: robot khepera, 3 links, 2 joints
Links:
- link chassis: geometry collision mesh filename=package://uned_kheperaiv_config/meshes/files/Empty_robot.dae scale=1.0 1.0 1.0; visual mesh filename=package://uned_kheperaiv_config/meshes/files/Empty_robot.dae scale=1.0 1.0 1.0
- link left_wheel: geometry collision mesh filename=package://uned_kheperaiv_config/meshes/files/wheel.dae scale=1.0 1.0 1.0; visual mesh filename=package://uned_kheperaiv_config/meshes/files/wheel.dae scale=1.0 1.0 1.0

File: uned_kheperaiv_config/urdf/khepera_simple.urdf (robot description, URDF)
Before this commit: robot khepera, 1 links, 0 joints
Links:
- link base_link: geometry collision mesh filename=package://uned_kheperaiv_config/meshes/files/Empty_robot.dae scale=1.0 1.0 1.0; visual mesh filename=package://uned_kheperaiv_config/meshes/files/Empty_robot.dae scale=1.0 1.0 1.0
